File: Hardware/Production/sparkfun-photon-redboard-Panel.brd (EAGLE design)
At the start: 176.8 x 151.1 mm, 218 parts, among them U1 WM-N-BM-14, U3 WM-N-BM-14, U5 WM-N-BM-14, U7 WM-N-BM-14

Commit message: Revised panel
Parts:
- added C49, C52, C57, C58, C59, C60, C61, C64, C69, C70, C71, C72, C73, C76, C81, C82, C83, C84, C85, C88, C93, C94, C95, C96: 0.1uF, SparkFun-Capacitors:0603-CAP
- added C50, C62, C74, C86: 10uF, SparkFun-Capacitors:EIA3216
- added C51, C63, C75, C87: 22uF, SparkFun-Capacitors:0805
- added C53, C54, C55, C56, C65, C66, C67, C68, C77, C78, C79, C80, C89, C90, C91, C92: 10uF, SparkFun-Capacitors:0603-CAP
- added D10, D12, D14, D16: RGB, SparkFun-LED:P-LCC-4-3
- added D11, D13, D15, D9: MBRA140, SparkFun-DiscreteSemi:SMA-DIODE
- added FID10, FID11, FID12, FID13, FID14, FID15, FID16, FID9: FIDUCIAL1X2, SparkFun-Aesthetics:FIDUCIAL-1X2
- added JP25, JP31, JP37, JP43: USB, SparkFun-Connectors:USB-B-MICRO-SMD_V03
- added JP26, JP32, JP38, JP44: POWER, SparkFun-Connectors:POWER_JACK_PTH_LOCK
- added JP27, JP33, JP39, JP45: ARDUINO_R3_NOISPLOCKING, sparkfun_photon_temp:ARDUINO_R3_NOISP_LOCKING
- added JP28, JP34, JP40, JP46: DNP, SparkFun-Connectors:2X10
- added JP29, JP35, JP41, JP47: DNP, SparkFun-Connectors:1X06
- added JP30, JP36, JP42, JP48: DNP, SparkFun-Connectors:1X02
- added LED10, LED12, LED14, LED16: RED, SparkFun-LED:LED-1206
- added LED11, LED13, LED15, LED9: BLUE, SparkFun-LED:LED-1206
- added LOGO13, LOGO16, LOGO19, LOGO22: SFE_LOGO_NAME_FLAME.2_INCH, SparkFun-Aesthetics:SFE_LOGO_NAME_FLAME_.2
- added LOGO14, LOGO17, LOGO20, LOGO23: OSHW-LOGOM, SparkFun-Aesthetics:OSHW-LOGO-M
- added LOGO15, LOGO18, LOGO21, LOGO24: SFE_LOGO_NAME_FLAME.4_INCH, SparkFun-Aesthetics:SFE_LOGO_NAME_FLAME_.4
- added R41, R42, R51, R52, R61, R62, R71, R72: 22, SparkFun-Resistors:0603-RES
- added R43, R53, R63, R73: 10K, SparkFun-Resistors:0603-RES
- added R44, R54, R64, R74: 100, SparkFun-Resistors:0603
- added R45, R55, R65, R75: 220, SparkFun-Resistors:0603
- added R46, R56, R66, R76: 100, SparkFun-Resistors:0603-RES
- added R47, R57, R67, R77: 300, SparkFun-Resistors:0603-RES
- added R48, R58, R68, R78: 1K, SparkFun-Resistors:0603-RES
- added R49, R59, R69, R79: 390, SparkFun-Resistors:0603-RES
- added R50, R60, R70, R80: 240, SparkFun-Resistors:0603-RES
- added S10, S12, S14, S16: MODE, SparkFun-Electromechanical:TACTILE-PTH
- added S11, S13, S15, S9: RESET, SparkFun-Electromechanical:TACTILE-PTH
- added SJ10, SJ12, SJ14, SJ16: D7-LED, SparkFun-Passives:PAD-JUMPER-2-NC_BY_TRACE_YES_SILK
- added SJ11, SJ13, SJ15, SJ9: PWR-LED, SparkFun-Passives:PAD-JUMPER-2-NC_BY_TRACE_YES_SILK
- added TP41, TP42, TP43, TP44, TP45, TP46, TP47, TP48, TP49, TP50, TP51, TP52, TP53, TP54, TP55, TP56, TP57, TP58, TP59, TP60, TP61, TP62, TP63, TP64, TP65, TP66, TP67, TP68, TP69, TP70, TP71, TP72, TP73, TP74, TP75, TP76, TP77, TP78, TP79, TP80: TEST-POINTTP_15TH_THRU, SparkFun-Passives:TP_15TH
- added U10, U12, U14, U16: (no value), SparkFun-PowerIC:SOT223
- added U11, U13, U15, U9: WM-N-BM-14, sparkfun_photon_temp:WM-N-BM-14
- moved C25 156.6 mm to (157.5, 20.3)
- moved C26 156.6 mm to (149.9, 14.0)
- moved C27 156.6 mm to (157.5, 22.2)
- moved C28 156.6 mm to (158.8, 47.0)
- moved C29 156.6 mm to (191.1, 9.53)
- moved C31 156.6 mm to (182.9, 19.7)
- moved C34 156.6 mm to (194.9, 34.3)
- moved C35 156.6 mm to (181.6, 19.7)
- moved FID5 156.6 mm to (146.1, 2.54)
- moved FID6 156.6 mm to (209.6, 48.3)
- moved JP13 156.6 mm to (146.9, 38.1)
- moved JP14 156.6 mm to (142.0, 7.62)
- moved JP15 156.6 mm to (144.8, 0.00)
- moved JP16 156.6 mm to (198.1, 43.2)
- moved JP17 156.6 mm to (207.0, 7.62)
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Connections:
- new net !MODE4: S10.3, U9.46
- new net !MODE5: S12.3, U11.46
- new net !MODE6: S14.3, U13.46
- new net !MODE7: S16.3, U15.46
- new net !RST4: C52.1, JP27.RESET@1, JP28.15, R43.1, S9.3, U9.34
- new net !RST5: C64.1, JP33.RESET@1, JP34.15, R53.1, S11.3, U11.34
- new net !RST6: C76.1, JP39.RESET@1, JP40.15, R63.1, S13.3, U13.34
- new net !RST7: C88.1, JP45.RESET@1, JP46.15, R73.1, S15.3, U15.34
- new net 3.3V4: C49.1, C51.1, C54.1, C55.1, C56.1, C58.1, C59.1, C60.1, D10.4, JP27.3.3V, JP28.1, R43.2, R48.2, R50.2, U10.2, U10.4, U9.2, U9.26, U9.27, U9.3, U9.5
- new net 3.3V5: C61.1, C63.1, C66.1, C67.1, C68.1, C70.1, C71.1, C72.1, D12.4, JP33.3.3V, JP34.1, R53.2, R58.2, R60.2, U11.2, U11.26, U11.27, U11.3, U11.5, U12.2, U12.4
- new net 3.3V6: C73.1, C75.1, C78.1, C79.1, C80.1, C82.1, C83.1, C84.1, D14.4, JP39.3.3V, JP40.1, R63.2, R68.2, R70.2, U13.2, U13.26, U13.27, U13.3, U13.5, U14.2, U14.4
- new net 3.3V7: C85.1, C87.1, C90.1, C91.1, C92.1, C94.1, C95.1, C96.1, D16.4, JP45.3.3V, JP46.1, R73.2, R78.2, R80.2, U15.2, U15.26, U15.27, U15.3, U15.5, U16.2, U16.4
- new net A12: JP27.A2, JP27.D10, U9.49
- new net A13: JP27.A1, U9.43
- new net A14: JP27.A0, U9.50
- new net A15: JP33.A2, JP33.D10, U11.49
- new net A16: JP33.A1, U11.43
- new net A17: JP33.A0, U11.50
- new net A18: JP39.A2, JP39.D10, U13.49
- new net A19: JP39.A1, U13.43
- new net A20: JP39.A0, U13.50
- new net A21: JP45.A2, JP45.D10, U15.49
- new net A22: JP45.A1, U15.43
- new net A23: JP45.A0, U15.50
- new net A3/SPI_SCK4: JP27.A3, JP27.D13, U9.22
- new net A3/SPI_SCK5: JP33.A3, JP33.D13, U11.22
- new net A3/SPI_SCK6: JP39.A3, JP39.D13, U13.22
- new net A3/SPI_SCK7: JP45.A3, JP45.D13, U15.22
- new net A4/SPI_MISO4: JP27.A4, JP27.D12, U9.21
- new net A4/SPI_MISO5: JP33.A4, JP33.D12, U11.21
- new net A4/SPI_MISO6: JP39.A4, JP39.D12, U13.21
- new net A4/SPI_MISO7: JP45.A4, JP45.D12, U15.21
- new net A5/SPI_MOSI4: JP27.A5, JP27.D11, U9.23
- new net A5/SPI_MOSI5: JP33.A5, JP33.D11, U11.23
- new net A5/SPI_MOSI6: JP39.A5, JP39.D11, U13.23
- new net A5/SPI_MOSI7: JP45.A5, JP45.D11, U15.23
- new net BTCX_RF_ACTIVE4: TP41.P$1, U9.57
- new net BTCX_RF_ACTIVE5: TP51.P$1, U11.57
- new net BTCX_RF_ACTIVE6: TP61.P$1, U13.57
- new net BTCX_RF_ACTIVE7: TP71.P$1, U15.57
- new net BTCX_STATUS4: TP43.P$1, U9.56
- new net BTCX_STATUS5: TP53.P$1, U11.56
- new net BTCX_STATUS6: TP63.P$1, U13.56
- new net BTCX_STATUS7: TP73.P$1, U15.56
- new net BTCX_TXCONF4: TP42.P$1, U9.58
- new net BTCX_TXCONF5: TP52.P$1, U11.58
- new net BTCX_TXCONF6: TP62.P$1, U13.58
- new net BTCX_TXCONF7: TP72.P$1, U15.58
- new net D+4: JP25.D+1, R42.1
- new net D+5: JP31.D+1, R52.1
- new net D+6: JP37.D+1, R62.1
- new net D+7: JP43.D+1, R72.1
- new net D-4: JP25.D-1, R41.1
- new net D-5: JP31.D-1, R51.1
- new net D-6: JP37.D-1, R61.1
- new net D-7: JP43.D-1, R71.1
- new net D0/SDA4: JP27.SDA, U9.36
- new net D0/SDA5: JP33.SDA, U11.36
- new net D0/SDA6: JP39.SDA, U13.36
- new net D0/SDA7: JP45.SDA, U15.36
- new net D1/SCL4: JP27.SCL, U9.35
- new net D1/SCL5: JP33.SCL, U11.35
- new net D1/SCL6: JP39.SCL, U13.35
- new net D1/SCL7: JP45.SCL, U15.35
- new net D3(JTAG_TRST)4: JP27.D3, JP28.3, U9.51
- new net D3(JTAG_TRST)5: JP33.D3, JP34.3, U11.51
- new net D3(JTAG_TRST)6: JP39.D3, JP40.3, U13.51
- new net D3(JTAG_TRST)7: JP45.D3, JP46.3, U15.51
- new net D4(JTAG_TDO)4: JP27.D4, JP28.13, U9.52
- new net D4(JTAG_TDO)5: JP33.D4, JP34.13, U11.52
- new net D4(JTAG_TDO)6: JP39.D4, JP40.13, U13.52
- new net D4(JTAG_TDO)7: JP45.D4, JP46.13, U15.52
- new net D5: JP27.D2, U9.45
- new net D5(JTAG_TDI)4: JP27.D5, JP28.5, U9.53
- new net D5(JTAG_TDI)5: JP33.D5, JP34.5, U11.53
- new net D5(JTAG_TDI)6: JP39.D5, JP40.5, U13.53
- new net D5(JTAG_TDI)7: JP45.D5, JP46.5, U15.53
- new net D6: JP33.D2, U11.45
- new net D6(JTAG_TCK)4: JP27.D6, JP28.9, U9.55
- new net D6(JTAG_TCK)5: JP33.D6, JP34.9, U11.55
- new net D6(JTAG_TCK)6: JP39.D6, JP40.9, U13.55
- new net D6(JTAG_TCK)7: JP45.D6, JP46.9, U15.55
- new net D7: JP39.D2, U13.45
- new net D7(JTAG_TMS)4: JP27.D7, JP28.7, R47.1, U9.54
- new net D7(JTAG_TMS)5: JP33.D7, JP34.7, R57.1, U11.54
- new net D7(JTAG_TMS)6: JP39.D7, JP40.7, R67.1, U13.54
- new net D7(JTAG_TMS)7: JP45.D7, JP46.7, R77.1, U15.54
- new net D8: JP45.D2, U15.45
- new net DAC4: JP27.D8, U9.24
- new net DAC5: JP33.D8, U11.24
- new net DAC6: JP39.D8, U13.24
- new net DAC7: JP45.D8, U15.24
- new net GND4: C49.2, C50.C, C51.2, C52.2, C53.2, C54.2, C55.2, C56.2, C57.2, C58.2, C59.2, C60.2, JP25.GND1, JP25.SHIELD1, JP25.SHIELD2, JP25.SHIELD3, JP26.GND, JP26.GNDBREAK, JP27.GND@1, JP27.GND@2, JP27.GND@3, JP28.10, JP28.11, JP28.12, JP28.14, JP28.16, JP28.18, JP28.20, JP28.4, JP28.6, JP28.8, JP30.1, R49.1, S10.1, S9.1, SJ10.1, SJ9.1, U9.1, U9.13, U9.15, U9.25, U9.28, U9.37, U9.39, U9.4, U9.59, U9.6, U9.65, U9.66, U9.67, U9.68, U9.69, U9.70, U9.71, U9.72, U9.73
- new net GND5: C61.2, C62.C, C63.2, C64.2, C65.2, C66.2, C67.2, C68.2, C69.2, C70.2, C71.2, C72.2, JP31.GND1, JP31.SHIELD1, JP31.SHIELD2, JP31.SHIELD3, JP32.GND, JP32.GNDBREAK, JP33.GND@1, JP33.GND@2, JP33.GND@3, JP34.10, JP34.11, JP34.12, JP34.14, JP34.16, JP34.18, JP34.20, JP34.4, JP34.6, JP34.8, JP36.1, R59.1, S11.1, S12.1, SJ11.1, SJ12.1, U11.1, U11.13, U11.15, U11.25, U11.28, U11.37, U11.39, U11.4, U11.59, U11.6, U11.65, U11.66, U11.67, U11.68, U11.69, U11.70, U11.71, U11.72, U11.73
- new net GND6: C73.2, C74.C, C75.2, C76.2, C77.2, C78.2, C79.2, C80.2, C81.2, C82.2, C83.2, C84.2, JP37.GND1, JP37.SHIELD1, JP37.SHIELD2, JP37.SHIELD3, JP38.GND, JP38.GNDBREAK, JP39.GND@1, JP39.GND@2, JP39.GND@3, JP40.10, JP40.11, JP40.12, JP40.14, JP40.16, JP40.18, JP40.20, JP40.4, JP40.6, JP40.8, JP42.1, R69.1, S13.1, S14.1, SJ13.1, SJ14.1, U13.1, U13.13, U13.15, U13.25, U13.28, U13.37, U13.39, U13.4, U13.59, U13.6, U13.65, U13.66, U13.67, U13.68, U13.69, U13.70, U13.71, U13.72, U13.73
- new net GND7: C85.2, C86.C, C87.2, C88.2, C89.2, C90.2, C91.2, C92.2, C93.2, C94.2, C95.2, C96.2, JP43.GND1, JP43.SHIELD1, JP43.SHIELD2, JP43.SHIELD3, JP44.GND, JP44.GNDBREAK, JP45.GND@1, JP45.GND@2, JP45.GND@3, JP46.10, JP46.11, JP46.12, JP46.14, JP46.16, JP46.18, JP46.20, JP46.4, JP46.6, JP46.8, JP48.1, R79.1, S15.1, S16.1, SJ15.1, SJ16.1, U15.1, U15.13, U15.15, U15.25, U15.28, U15.37, U15.39, U15.4, U15.59, U15.6, U15.65, U15.66, U15.67, U15.68, U15.69, U15.70, U15.71, U15.72, U15.73
- new net MCU_USB_D+4: R42.2, U9.61
- new net MCU_USB_D+5: R52.2, U11.61
- new net MCU_USB_D+6: R62.2, U13.61
- new net MCU_USB_D+7: R72.2, U15.61
- new net MCU_USB_D-4: R41.2, U9.62
- new net MCU_USB_D-5: R51.2, U11.62
- new net MCU_USB_D-6: R61.2, U13.62
- new net MCU_USB_D-7: R71.2, U15.62
- new net N$37: R49.2, R50.1, U10.1
- new net N$38: D10.2, R46.1
- new net N$39: D10.1, R45.1
- new net N$40: LED9.A, R47.2
- new net N$41: LED10.A, R48.1
- new net N$42: TP50.P$1, U9.33
- new net N$43: LED10.C, SJ9.2
- new net N$44: LED9.C, SJ10.2
- new net N$45: D10.3, R44.1
- new net N$46: R59.2, R60.1, U12.1
- new net N$47: D12.2, R56.1
- new net N$48: D12.1, R55.1
- new net N$49: LED11.A, R57.2
- new net N$50: LED12.A, R58.1
- new net N$51: TP60.P$1, U11.33
- new net N$52: LED12.C, SJ11.2
- new net N$53: LED11.C, SJ12.2
- new net N$54: D12.3, R54.1
- new net N$55: R69.2, R70.1, U14.1
- new net N$56: D14.2, R66.1
- new net N$57: D14.1, R65.1
- new net N$58: LED13.A, R67.2
- new net N$59: LED14.A, R68.1
- new net N$60: TP70.P$1, U13.33
- new net N$61: LED14.C, SJ13.2
- new net N$62: LED13.C, SJ14.2
- new net N$63: D14.3, R64.1
- new net N$64: R79.2, R80.1, U16.1
- new net N$65: D16.2, R76.1
- new net N$66: D16.1, R75.1
- new net N$67: LED15.A, R77.2
- new net N$68: LED16.A, R78.1
- new net N$69: TP80.P$1, U15.33
- new net N$70: LED16.C, SJ15.2
- new net N$71: LED15.C, SJ16.2
- new net N$72: D16.3, R74.1
- new net RGB_BLUE4: R44.2, U9.31
- new net RGB_BLUE5: R54.2, U11.31
- new net RGB_BLUE6: R64.2, U13.31
- new net RGB_BLUE7: R74.2, U15.31
- new net RGB_GREEN4: R46.2, U9.32
- new net RGB_GREEN5: R56.2, U11.32
- new net RGB_GREEN6: R66.2, U13.32
- new net RGB_GREEN7: R76.2, U15.32
- new net RGB_RED4: R45.2, U9.29
- new net RGB_RED5: R55.2, U11.29
- new net RGB_RED6: R65.2, U13.29
- new net RGB_RED7: R75.2, U15.29
- new net RX4: JP27.D0, U9.63
- new net RX5: JP33.D0, U11.63
- new net RX6: JP39.D0, U13.63
- new net RX7: JP45.D0, U15.63
- new net SPARE25: JP29.6, U9.40
- new net SPARE26: JP29.5, U9.41
- new net SPARE27: JP29.4, U9.42
- new net SPARE28: JP29.3, U9.44
- new net SPARE29: JP29.2, U9.47
- new net SPARE30: JP29.1, U9.48
- new net SPARE31: JP35.6, U11.40
- new net SPARE32: JP35.5, U11.41
- new net SPARE33: JP35.4, U11.42
- new net SPARE34: JP35.3, U11.44
- new net SPARE35: JP35.2, U11.47
- new net SPARE36: JP35.1, U11.48
- new net SPARE37: JP41.6, U13.40
- new net SPARE38: JP41.5, U13.41
- new net SPARE39: JP41.4, U13.42
- new net SPARE40: JP41.3, U13.44
- new net SPARE41: JP41.2, U13.47
- new net SPARE42: JP41.1, U13.48
- new net SPARE43: JP47.6, U15.40
- new net SPARE44: JP47.5, U15.41
- new net SPARE45: JP47.4, U15.42
- new net SPARE46: JP47.3, U15.44
- new net SPARE47: JP47.2, U15.47
- new net SPARE48: JP47.1, U15.48
- new net TX4: JP27.D1, U9.64
- new net TX5: JP33.D1, U11.64
- new net TX6: JP39.D1, U13.64
- new net TX7: JP45.D1, U15.64
- new net VBAT4: C53.1, C57.1, JP30.2, U9.38
- new net VBAT5: C65.1, C69.1, JP36.2, U11.38
- new net VBAT6: C77.1, C81.1, JP42.2, U13.38
- new net VBAT7: C89.1, C93.1, JP48.2, U15.38
- new net VIN4: C50.A, D9.C, JP26.PWR, JP27.VIN, U10.3
- new net VIN5: C62.A, D11.C, JP32.PWR, JP33.VIN, U12.3
- new net VIN6: C74.A, D13.C, JP38.PWR, JP39.VIN, U14.3
- new net VIN7: C86.A, D15.C, JP44.PWR, JP45.VIN, U16.3
- new net VUSB4: D9.A, JP25.VBUS1, JP27.5V
- new net VUSB5: D11.A, JP31.VBUS1, JP33.5V
- new net VUSB6: D13.A, JP37.VBUS1, JP39.5V
- new net VUSB7: D15.A, JP43.VBUS1, JP45.5V
- new net WKP4: JP27.D9, U9.30
- new net WKP5: JP33.D9, U11.30
- new net WKP6: JP39.D9, U13.30
- new net WKP7: JP45.D9, U15.30
- new net WL_JTAG_TCK4: TP45.P$1, U9.17
- new net WL_JTAG_TCK5: TP55.P$1, U11.17
- new net WL_JTAG_TCK6: TP65.P$1, U13.17
- new net WL_JTAG_TCK7: TP75.P$1, U15.17
- new net WL_JTAG_TDI4: TP44.P$1, U9.16
- new net WL_JTAG_TDI5: TP54.P$1, U11.16
- new net WL_JTAG_TDI6: TP64.P$1, U13.16
- new net WL_JTAG_TDI7: TP74.P$1, U15.16
- new net WL_JTAG_TDO4: TP48.P$1, U9.20
- new net WL_JTAG_TDO5: TP58.P$1, U11.20
- new net WL_JTAG_TDO6: TP68.P$1, U13.20
- new net WL_JTAG_TDO7: TP78.P$1, U15.20
- new net WL_JTAG_TMS4: TP47.P$1, U9.19
- new net WL_JTAG_TMS5: TP57.P$1, U11.19
- new net WL_JTAG_TMS6: TP67.P$1, U13.19
- new net WL_JTAG_TMS7: TP77.P$1, U15.19
- new net WL_JTAG_TRST4: TP46.P$1, U9.18
- new net WL_JTAG_TRST5: TP56.P$1, U11.18
- new net WL_JTAG_TRST6: TP66.P$1, U13.18
- new net WL_JTAG_TRST7: TP76.P$1, U15.18
- new net WL_SLEEP_CLK4: TP49.P$1, U9.60
- new net WL_SLEEP_CLK5: TP59.P$1, U11.60
- new net WL_SLEEP_CLK6: TP69.P$1, U13.60
- new net WL_SLEEP_CLK7: TP79.P$1, U15.60
Routing:
- net 3.3V7: track 0.00 -> 157.3 mm, vias 0 -> 15
- net 3.3V6: track 0.00 -> 157.3 mm, vias 0 -> 15
- net 3.3V5: track 0.00 -> 157.3 mm, vias 0 -> 15
- net 3.3V4: track 0.00 -> 157.3 mm, vias 0 -> 15
- net !RST5: track 0.00 -> 120.3 mm, vias 0 -> 5
- net !RST7: track 0.00 -> 120.3 mm, vias 0 -> 5
- net !RST6: track 0.00 -> 120.3 mm, vias 0 -> 5
- net !RST4: track 0.00 -> 120.3 mm, vias 0 -> 5
- net D7(JTAG_TMS)7: track 0.00 -> 86.6 mm, vias 0 -> 5
- net D7(JTAG_TMS)6: track 0.00 -> 86.6 mm, vias 0 -> 5
- net D7(JTAG_TMS)5: track 0.00 -> 86.6 mm, vias 0 -> 5
- net D7(JTAG_TMS)4: track 0.00 -> 86.6 mm, vias 0 -> 5
- net VIN6: track 0.00 -> 83.8 mm, vias 0 -> 4
- net VIN5: track 0.00 -> 83.8 mm, vias 0 -> 4
- net VIN4: track 0.00 -> 83.8 mm, vias 0 -> 4
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- added copper zone on layer 1, net 3.3V4
- added copper zone on layer 16, net 3.3V4
- added copper zone on layer 1, net 3.3V5
- added copper zone on layer 16, net 3.3V5
- added copper zone on layer 1, net 3.3V6
- added copper zone on layer 16, net 3.3V6
- added copper zone on layer 1, net 3.3V7
- added copper zone on layer 16, net 3.3V7
- added copper zone on layer 1, net GND4
- added copper zone on layer 16, net GND4
- added copper zone on layer 1, net GND5
- added copper zone on layer 16, net GND5
- added copper zone on layer 1, net GND6
- added copper zone on layer 16, net GND6
- added copper zone on layer 1, net GND7
- added copper zone on layer 16, net GND7
Other:
- board size 176.8 x 151.1 mm -> 311.1 x 135.9 mm
